File: hardware/domo_pool_hard/_autosave-domo_pool_hard.sch (KiCad schematic (older format))
At the start: 18 parts

Commit message: schematic
Parts:
- added J?: Screw_Terminal_01x04, symbol Connector:Screw_Terminal_01x04
- added Q?: TIP120, Package_TO_SOT_THT:TO-220-3_Vertical, symbol Transistor_BJT:TIP120
Connections:
- net +12V: now also J?.1 (Pin_1), J?.2 (Pin_2)
- net GND: now also J?.3 (Pin_3), J?.4 (Pin_4)
Changed lines of the file:
@@
 Text GLabel 9700 5750 0    50   Input ~ 0
 44
+$Comp
+L Connector:Screw_Terminal_01x04 J?
+U 1 1 612E70E1
+P 12450 1300
+F 0 "J?" H 12530 1292 50  0000 L CNN
+F 1 "Screw_Terminal_01x04" H 12530 1201 50  0000 L CNN
+F 2 "" H 12450 1300 50  0001 C CNN
+F 3 "~" H 12450 1300 50  0001 C CNN
+	1    12450 1300
+	1    0    0    -1
+$EndComp
+$Comp
+L power:+12V #PWR?
+U 1 1 612E975F
+P 12100 1050
+F 0 "#PWR?" H 12100 900 50  0001 C CNN
+F 1 "+12V" H 12115 1223 50  0000 C CNN
+F 2 "" H 12100 1050 50  0001 C CNN
+F 3 "" H 12100 1050 50  0001 C CNN
+	1    12100 1050
+	1    0    0    -1
+$EndComp
+$Comp
+L power:GND #PWR?
+U 1 1 612E9E12
+P 12100 1700
+F 0 "#PWR?" H 12100 1450 50  0001 C CNN
+F 1 "GND" H 12105 1527 50  0000 C CNN
+F 2 "" H 12100 1700 50  0001 C CNN
+F 3 "" H 12100 1700 50  0001 C CNN
+	1    12100 1700
+	1    0    0    -1
+$EndComp
+Wire Wire Line
+	12100 1700 12100 1500
+Wire Wire Line
+	12100 1400 12250 1400
+Wire Wire Line
+	12250 1500 12100 1500
+Connection ~ 12100 1500
+Wire Wire Line
+	12100 1500 12100 1400
+Wire Wire Line
+	12250 1200 12100 1200
+Wire Wire Line
+	12100 1200 12100 1050
+Wire Wire Line
+	12250 1300 12100 1300
+Wire Wire Line
+	12100 1300 12100 1200
+Connection ~ 12100 1200
+$Comp
+L Transistor_BJT:TIP120 Q?
+U 1 1 61336F93
+P 8650 9100
+F 0 "Q?" H 8857 9146 50  0000 L CNN
+F 1 "TIP120" H 8857 9055 50  0000 L CNN
+F 2 "Package_TO_SOT_THT:TO-220-3_Vertical" H 8850 9025 50  0001 L CIN
+F 3 "https://www.onsemi.com/pub/Collateral/TIP120-D.PDF" H 8650 9100 50  0001 L CNN
+	1    8650 9100
+	1    0    0    -1
+$EndComp
 $EndSCHEMATC
